File: pcb1/pcb1.kicad_pcb (KiCad board)
At the start: 2 copper layers, 80 x 125 mm, 19 parts, among them J1 Input, J2 Output, Q1 IRFZ44N, U1 LM358

Commit message: new schema
Parts:
- added D2: LED, LED_THT:LED_D3.0mm_Clear, F.Cu at (91.4, 97.8)
- added R2: 1k, Resistor_THT:R_Axial_DIN0207_L6.3mm_D2.5mm_P10.16mm_Horizontal, F.Cu at (85.6, 108.7)
- moved D1 4.32 mm to (103.1, 105.9)
- moved R1 4.32 mm to (89.9, 105.9)
- moved REF** 0.63 mm to (47.8, 39.6)
- moved REF** 0.54 mm to (116.6, 39.6)
- moved REF** 0.46 mm to (116.6, 153.4)
Routing:
- net Net-(Q1-S): track 168.6 -> 98.3 mm, vias 0 -> 2
- net /load-: track 163.4 -> 180.5 mm
- net Net-(Q1-G): track 89.7 -> 80.3 mm
- net GND: track 128.0 -> 123.6 mm
- net Net-(D2-A): track 0.00 -> 3.62 mm
- net VCC: track 242.5 -> 241.8 mm
- added copper zone on F.Cu, net (none)
- removed copper zone on F.Cu, net GND

Commit message: fix nmos pin order
Parts:
- F1: value 10A -> 15A
- RSense1: value 0R02 -> 0R01
- Rb1: value 130R -> 56R
- moved R4 35.9 mm to (112.5, 91.7), turned to 180 degrees
- moved R2 24.1 mm to (107.2, 98.0), turned to 180 degrees
- moved D2 0.80 mm to (90.7, 98.0), turned to 0 degrees
Connections:
- Q1 pad 1: /load- -> Net-(Q1-G)
- Q1 pad 2: Net-(Q1-G) -> /load-
- U1 pad 5: unconnected-(U1B-+-Pad5) -> GND
- U1 pad 6: unconnected-(U1B---Pad6) -> GND
Routing:
- net GND: track 123.6 -> 161.5 mm
- net Net-(Q1-G): track 80.3 -> 63.5 mm, vias 2 -> 0
- net /load-: track 180.5 -> 166.5 mm
- net VCC: track 241.8 -> 248.0 mm
- net Net-(Q1-S): track 98.3 -> 100.3 mm
- net Net-(D1-K): track 9.71 -> 11.0 mm

Commit message: remove fuse
Parts:
- removed F1: 15A, Fuse:Fuseholder_Clip-5x20mm_Eaton_1A5601-01_Inline_P20.80x6.76mm_D1.70mm_Horizontal
Connections:
- J1 pad 1: Net-(J1-Pin_1) -> VCC
Routing:
- net Net-(J1-Pin_1): track 18.9 -> 0.00 mm
- net VCC: track 248.0 -> 243.9 mm
