File: pcb2/pcb1.kicad_sch (KiCad schematic)
At the start: 18 parts, among them Q1 IRFZ44N, U1 LM358, U2 NE555P, X1 Input, X2 Output

Commit message: make a board of with ne555
Parts:
- added C6: 100nf, Capacitor_THT:C_Rect_L7.2mm_W6.0mm_P5.00mm, symbol Device:C
- added R8: 10R, Resistor_THT:R_Axial_DIN0207_L6.3mm_D2.5mm_P10.16mm_Horizontal, symbol Device:R
- C4, C5: footprint (none) -> Capacitor_THT:C_Rect_L7.2mm_W6.0mm_P5.00mm
Connections:
- net GND: now also C6.2
- net VCC: now also C6.1
- net at Q1.1 (G), R4.2: now also R8.1; no longer U1.7
- new net: R8.2, U1.7
Changed lines of the file:
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@@
 	(paper "A4")
 	(junction
+		(at 102.87 86.36)
+		(diameter 0)
+		(color 0 0 0 0)
+	)
+	(junction
+		(at 58.42 80.01)
+		(diameter 0)
+		(color 0 0 0 0)
+	)
+	(junction
 		(at 58.42 95.25)
 		(diameter 0)
@@
 	)
 	(junction
-		(at 74.93 52.07)
+		(at 44.45 52.07)
 		(diameter 0)
 		(color 0 0 0 0)
@@
 		(color 0 0 0 0)
 	)
+	(junction
+		(at 58.42 55.88)
+		(diameter 0)
+		(color 0 0 0 0)
+	)
 	(no_connect
 		(at 77.47 74.93)
@@
 	(wire
 		(pts
-			(xy 102.87 83.82) (xy 114.3 83.82)
+			(xy 102.87 86.36) (xy 114.3 86.36)
 		)
 		(stroke
@@
 	(wire
 		(pts
+			(xy 58.42 80.01) (xy 58.42 95.25)
+		)
+		(stroke
+			(width 0)
+			(type default)
+		)
+	)
+	(wire
+		(pts
 			(xy 87.63 64.77) (xy 87.63 57.15)
 		)
@@
 	(wire
 		(pts
-			(xy 166.37 59.69) (xy 166.37 77.47)
+			(xy 48.26 80.01) (xy 58.42 80.01)
+		)
+		(stroke
+			(width 0)
+			(type default)
+		)
+	)
+	(wire
+		(pts
+			(xy 166.37 59.69) (xy 166.37 64.77)
 		)
 		(stroke
@@
 	(wire
 		(pts
-			(xy 114.3 83.82) (xy 114.3 57.15)
+			(xy 114.3 86.36) (xy 114.3 57.15)
+		)
+		(stroke
+			(width 0)
+			(type default)
+		)
+	)
+	(wire
+		(pts
+			(xy 166.37 72.39) (xy 166.37 77.47)
 		)
 		(stroke
@@
 	(wire
 		(pts
+			(xy 48.26 55.88) (xy 58.42 55.88)
+		)
+		(stroke
+			(width 0)
+			(type default)
+		)
+	)
+	(wire
+		(pts
 			(xy 102.87 62.23) (xy 102.87 52.07)
 		)
@@
 	(wire
 		(pts
-			(xy 58.42 52.07) (xy 58.42 59.69)
+			(xy 58.42 52.07) (xy 58.42 55.88)
 		)
 		(stroke
@@
 	(wire
 		(pts
+			(xy 102.87 86.36) (xy 102.87 87.63)
+		)
+		(stroke
+			(width 0)
+			(type default)
+		)
+	)
+	(wire
+		(pts
+			(xy 48.26 71.12) (xy 48.26 80.01)
+		)
+		(stroke
+			(width 0)
+			(type default)
+		)
+	)
+	(wire
+		(pts
 			(xy 121.92 86.36) (xy 121.92 80.01)
 		)
@@
 	(wire
 		(pts
-			(xy 58.42 74.93) (xy 58.42 95.25)
+			(xy 58.42 74.93) (xy 58.42 80.01)
 		)
 		(stroke
@@
 	(wire
 		(pts
-			(xy 102.87 83.82) (xy 102.87 87.63)
+			(xy 102.87 83.82) (xy 102.87 86.36)
 		)
 		(stroke
@@
 	(wire
 		(pts
+			(xy 48.26 63.5) (xy 48.26 55.88)
+		)
+		(stroke
+			(width 0)
+			(type default)
+		)
+	)
+	(wire
+		(pts
 			(xy 228.6 72.39) (xy 237.49 72.39)
 		)
@@
 		)
 	)
+	(wire
+		(pts
+			(xy 58.42 55.88) (xy 58.42 59.69)
+		)
+		(stroke
+			(width 0)
+			(type default)
+		)
+	)
 	(label "load-"
 		(at 237.49 46.99 0)
@@
 			)
 		)
-		(property "Footprint" ""
+		(property "Footprint" "Capacitor_THT:C_Rect_L7.2mm_W6.0mm_P5.00mm"
 			(at 73.3552 95.25 0)
 			(hide yes)
@@
 	(symbol
 		(lib_id "power:VCC")
-		(at 74.93 52.07 0)
+		(at 44.45 52.07 0)
 		(unit 1)
 		(body_style 1)
@@
 		(fields_autoplaced yes)
 		(property "Reference" "#PWR02"
-			(at 74.93 55.88 0)
+			(at 44.45 55.88 0)
 			(hide yes)
 			(show_name no)
@@
 		)
 		(property "Value" "VCC"
-			(at 74.93 46.99 0)
+			(at 44.45 46.99 0)
 			(show_name no)
 			(do_not_autoplace no)
@@
 		)
 		(property "Footprint" ""
-			(at 74.93 52.07 0)
+			(at 44.45 52.07 0)
 			(hide yes)
 			(show_name no)
@@
 		)
 		(property "Datasheet" ""
-			(at 74.93 52.07 0)
+			(at 44.45 52.07 0)
 			(hide yes)
 			(show_name no)
@@
 		)
 		(property "Description" "Power symbol creates a global label with name \"VCC\""
-			(at 74.93 52.07 0)
+			(at 44.45 52.07 0)
 			(hide yes)
 			(show_name no)
@@
 	)
 	(symbol
+		(lib_id "Device:C")
+		(at 48.26 67.31 0)
+		(unit 1)
+		(body_style 1)
+		(exclude_from_sim no)
+		(in_bom yes)
+		(on_board yes)
+		(in_pos_files yes)
+		(dnp no)
+		(fields_autoplaced yes)
+		(property "Reference" "C6"
+			(at 52.07 66.0399 0)
+			(show_name no)
+			(do_not_autoplace no)
+			(effects
+				(font
+					(size 1.27 1.27)
+				)
+				(justify left)
+			)
+		)
+		(property "Value" "100nf"
+			(at 52.07 68.5799 0)
+			(show_name no)
+			(do_not_autoplace no)
+			(effects
+				(font
+					(size 1.27 1.27)
+				)
+				(justify left)
+			)
+		)
+		(property "Footprint" "Capacitor_THT:C_Rect_L7.2mm_W6.0mm_P5.00mm"
+			(at 49.2252 71.12 0)
+			(hide yes)
+			(show_name no)
+			(do_not_autoplace no)
+			(effects
+				(font
+					(size 1.27 1.27)
+				)
+			)
+		)
+		(property "Datasheet" ""
+			(at 48.26 67.31 0)
+			(hide yes)
+			(show_name no)
+			(do_not_autoplace no)
+			(effects
+				(font
+					(size 1.27 1.27)
+				)
+			)
+		)
+		(property "Description" "Unpolarized capacitor"
+			(at 48.26 67.31 0)
+			(hide yes)
+			(show_name no)
+			(do_not_autoplace no)
+			(effects
+				(font
+					(size 1.27 1.27)
+				)
+			)
+		)
+		(pin "1"
+		)
+		(pin "2"
+		)
+		(instances
+			(project "pcb1"
+				(path "/0501d330-5f5d-44b9-93b3-0b7cc442c6a9"
+					(reference "C6")
+					(unit 1)
+				)
+			)
+		)
+	)
+	(symbol
 		(lib_id "Timer:NE555P")
 		(at 87.63 74.93 0)
@@
 	)
 	(symbol
-		(lib_id "power:GND")
-		(at 87.63 95.25 0)
+		(lib_id "Device:R")
+		(at 166.37 68.58 180)
 		(unit 1)
 		(body_style 1)
@@
 		(dnp no)
 		(fields_autoplaced yes)
-		(property "Reference" "#PWR03"
-			(at 87.63 101.6 0)
-			(hide yes)
+		(property "Reference" "R8"
+			(at 168.91 67.3099 0)
 			(show_name no)
 			(do_not_autoplace no)
@@
 					(size 1.27 1.27)
 				)
+				(justify right)
 			)
 		)
-		(property "Value" "GND"
-			(at 87.63 100.33 0)
+		(property "Value" "10R"
+			(at 168.91 69.8499 0)
 			(show_name no)
 			(do_not_autoplace no)
@@
 					(size 1.27 1.27)
 				)
+				(justify right)
 			)
 		)
-		(property "Footprint" ""
-			(at 87.63 95.25 0)
+		(property "Footprint" "Resistor_THT:R_Axial_DIN0207_L6.3mm_D2.5mm_P10.16mm_Horizontal"
+			(at 168.148 68.58 90)
 			(hide yes)
 			(show_name no)
@@
 		)
 		(property "Datasheet" ""
-			(at 87.63 95.25 0)
+			(at 166.37 68.58 0)
 			(hide yes)
 			(show_name no)
@@
 			)
 		)
-		(property "Description" "Power symbol creates a global label with name \"GND\" , ground"
-			(at 87.63 95.25 0)
+		(property "Description" "Resistor"
+			(at 166.37 68.58 0)
 			(hide yes)
 			(show_name no)
@@
 			)
 		)
+		(property "KiLib_Generator" "resistor/THT"
+			(at 166.37 68.58 0)
+			(hide yes)
+			(show_name no)
+			(do_not_autoplace no)
+			(effects
+				(font
+					(size 1.27 1.27)
+				)
+			)
+		)
+		(pin "2"
+		)
 		(pin "1"
 		)
@@
 			(project "pcb1"
 				(path "/0501d330-5f5d-44b9-93b3-0b7cc442c6a9"
-					(reference "#PWR03")
+					(reference "R8")
 					(unit 1)
 				)
@@
 			)
 		)
-		(property "Footprint" ""
+		(property "Footprint" "Capacitor_THT:C_Rect_L7.2mm_W6.0mm_P5.00mm"
 			(at 103.8352 95.25 0)
 			(hide yes)

Commit message: add zener to stability
Parts:
- added D1: 8V2, Diode_THT:D_DO-35_SOD27_P7.62mm_Horizontal, symbol Device:D_Zener
- added R1: 760R, Resistor_THT:R_Axial_DIN0207_L6.3mm_D2.5mm_P10.16mm_Horizontal, symbol Device:R
- R6: value 100R -> 10R
Connections:
- net GND: now also D1.2 (A)
- net VCC: now also R1.1
- net at C4.1, U2.5 (CONT): now also D1.1 (K), R1.2
Other:
- moved on the sheet: C4, X2

Commit message: ready to print
Parts:
- C4: footprint Capacitor_THT:C_Rect_L7.2mm_W6.0mm_P5.00mm -> Capacitor_THT:C_Rect_L7.2mm_W3.5mm_P5.00mm_FKS2_FKP2_MKS2_MKP2
- C5: footprint Capacitor_THT:C_Rect_L7.2mm_W6.0mm_P5.00mm -> Capacitor_THT:C_Rect_L7.0mm_W3.5mm_P5.00mm
- C6: footprint Capacitor_THT:C_Rect_L7.2mm_W6.0mm_P5.00mm -> Capacitor_THT:C_Rect_L9.0mm_W3.3mm_P7.50mm_MKT
- R1: value 760R -> 680R
Changed lines of the file:
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@@
 			)
 		)
-		(property "Footprint" "Capacitor_THT:C_Rect_L7.2mm_W6.0mm_P5.00mm"
+		(property "Footprint" "Capacitor_THT:C_Rect_L7.2mm_W3.5mm_P5.00mm_FKS2_FKP2_MKS2_MKP2"
 			(at 77.1652 93.98 0)
 			(hide yes)
@@
 			)
 		)
-		(property "Value" "760R"
+		(property "Value" "680R"
 			(at 71.12 58.4199 0)
 			(show_name no)
@@
 			)
 		)
-		(property "Footprint" "Capacitor_THT:C_Rect_L7.2mm_W6.0mm_P5.00mm"
+		(property "Footprint" "Capacitor_THT:C_Rect_L9.0mm_W3.3mm_P7.50mm_MKT"
 			(at 49.2252 71.12 0)
 			(hide yes)
@@
 			)
 		)
-		(property "Footprint" "Capacitor_THT:C_Rect_L7.2mm_W6.0mm_P5.00mm"
+		(property "Footprint" "Capacitor_THT:C_Rect_L7.0mm_W3.5mm_P5.00mm"
 			(at 103.8352 95.25 0)
 			(hide yes)
